File: cad/goldfish.kicad_pcb (KiCad board)
At the start: 2 copper layers, 17.8 x 33 mm, 25 parts, among them J1 USB-C, J2 01x02, J3 01x12, J4 01x12, J5 01x05, U1 ATmega32U4, X1 16MHz

Commit message: removed goldfish silk
Parts:
- removed G***: LOGO, fish:fish-cu
Other:
- net class Default removed
- net class PWR removed
- board text removed: "Rev.C"
- board text removed: "USB"
- board text removed: "goldfish"
- board text removed: "∂r_∂erivative"
