File: cad/goldfish.kicad_pcb (KiCad board)
At the start: 2 copper layers, 17.8 x 33 mm, 24 parts, among them J1 USB-C, J2 01x02, J3 01x12, J4 01x12, J5 01x05, U1 ATmega32U4, X1 16MHz

Commit message: adding silks
Parts:
- added G***: LOGO, fmkc:fmkc_logo, B.Cu at (30.0, 40.0)

Commit message: tyty-c addition test
Parts:
- added G***: LOGO, fmkc:tyty-c, B.Cu at (29.9, 41.2)
- moved G*** 15.1 mm to (14.9, 40.0)

Commit message: idk plotted things, pcb artworks etc random work, should prolly gitignore plot-folder but cba :D
Parts:
- removed the G*** at (29.9, 41.2)
- removed the G*** at (14.9, 40.0)
- added G***: LOGO, fmkc:pikkuinen, B.Cu at (30.0, 41.3)
- U1: footprint Package_DFN_QFN:QFN-44-1EP_7x7mm_P0.5mm_EP5.2x5.2mm -> fmkc:QFN-44-1EP_7x7mm_P0.5mm_EP5.2x5.2mm_FORK
Other:
- rule pad_to_mask_clearance: 0.2 -> 0
